Commit message: Final rover TP task submission

File: rover_ws/install/gazebo/share/gazebo/model/rover.xacro (robot description, xacro)
@@ -1,8 +1,24 @@
 <?xml version = "1.0"?>
 <robot xmlns:xacro="http://www.ros.org/wiki/xacro" name= "rover">
+<xacro:property name = "base_link_x" value = "0.5"/>
+<xacro:property name = "base_link_y" value = "1"/>
+<xacro:property name = "base_link_z" value = "0.25"/>
+<xacro:property name = "wheel_link_radius" value = "0.15"/>
+<xacro:property name = "wheel_link_length" value = "0.05"/>
+<xacro:property name = "wheel_link_z" value = "-0.05"/>
+<xacro:property name = "density" value = "2710.0"/>
+<xacro:property name = "pi_constant" value = "3.14159"/>
+<xacro:property name = "base_mass" value = "${density*base_link_x*base_link_y*base_link_z}"/>
+<xacro:property name = "wheel_mass" value = "${density*pi_constant*wheel_link_radius*wheel_link_radius*wheel_link_length}"/>
+<xacro:property name = "Iz_wheel" value = "${0.5*wheel_mass*wheel_link_radius*wheel_link_radius}"/>
+<xacro:property name = "I_wheel" value = "${(1/12)*wheel_mass*(3*wheel_link_radius*wheel_link_radius+wheel_link_length*wheel_link_length)}"/>
+<xacro:macro name = "inertial_wheel">
+<inertial>
+<origin rpy = "0 0 0" xyz = "0 0 0"/>
+<mass value = "${wheel_mass}"/>
+<inertia ixx = "${I_wheel}" ixy = "0" ixz = "0" iyy = "${I_wheel}" iyz = "0" izz = "${Iz_wheel}" />
+</inertial>
+</xacro:macro>
 <xacro:include filename="$(find gazebo)/model/rover.gazebo"/>
-<xacro:property name = "body_link_y_dim" value = "1"/>
-<xacro:property name = "wheel_link_length" value = "0.05"/>
-<xacro:property name = "wheel_link_radius" value = "0.15"/>
 <material name = "black">
     <color rgba = " 0 0 0 1"/>
@@ -29,5 +45,5 @@
         <visual>
             <geometry>
-                <box size = " 0.5 1 0.25"/>
+                <box size = "${base_link_x} ${base_link_y} ${base_link_z}"/>
             </geometry>
             <origin xyz = " 0 0 0.125" rpy = "0 0 0"/>
@@ -36,5 +52,5 @@
     <collision>
             <geometry>
-                <box size = " 0.5 1 0.25"/>
+                <box size = "${base_link_x} ${base_link_y} ${base_link_z}"/>
             </geometry>
             <origin xyz = " 0 0 0.125" rpy = "0 0 0"/>
@@ -42,6 +58,10 @@
     <inertial>
         <origin xyz = " 0 0 0.125" rpy = "0 0 0"/>
-        <mass value= "2"/>
-        <inertia ixx = "100" ixy = "0" ixz = "0" iyy = "100" izz = "100" iyz = "0"/>
+        <mass value= "${base_mass}"/>
+        <inertia ixx = "${(1/12)*base_mass*(base_link_y*base_link_y+base_link_z*base_link_z)}"
+        ixy = "0" ixz = "0"
+        iyy = "${(1/12)*base_mass*(base_link_x*base_link_x+base_link_z*base_link_z)}"
+        izz = "${(1/12)*base_mass*(base_link_y*base_link_y+base_link_x*base_link_x)}"
+        iyz = "0"/>
     </inertial>
     </link>
@@ -49,5 +69,5 @@
     <parent link = "base_link"/>
     <child link = "left_front_link"/>
-    <origin xyz = "0.275 0.45 0" rpy = "0 0 0" />
+    <origin xyz = "0.275 ${-base_link_y/2-wheel_link_length/2} ${wheel_link_z}" rpy = "0 0 0" />
     <axis xyz ="1 0 0"/>
     <limit effort = "1000" velocity = "1000"/>
@@ -57,25 +77,21 @@
         <visual>
             <geometry>
-                <cylinder radius = "0.15" length = "0.05"/>
-            </geometry>
-            <origin xyz = " 0 0 0" rpy = "0 1.57 0"/>
+                <cylinder radius = "${wheel_link_radius}" length = "${wheel_link_length}"/>
+            </geometry>
+            <origin xyz = " 0 0 0" rpy = "0 1.570795 0"/>
             <material name = "white"/>
         </visual>
     <collision>
             <geometry>
-                <cylinder radius = "0.15" length = "0.05"/>
-            </geometry>
-            <origin xyz = " 0 0 0" rpy = "0 1.57 0"/>
-    </collision>
-    <inertial>
-         <origin xyz = " 0 0 0" rpy = "0 1.57 0"/>
-        <mass value= "0.25"/>
-        <inertia ixx = "100" ixy = "0" ixz = "0" iyy = "100" izz = "100" iyz = "0"/>
-    </inertial>
+                 <cylinder radius = "${wheel_link_radius}" length = "${wheel_link_length}"/>
+            </geometry>
+            <origin xyz = " 0 0 0" rpy = "0 1.570795 0"/>
+    </collision>
+<xacro:inertial_wheel/>
     </link>
 <joint name = "right_front_wheel_joint" type = "continuous">
     <parent link = "base_link"/>
     <child link = "right_front_link"/>
-    <origin xyz = "-0.275 0.45 0" rpy = "0 0 0" />
+    <origin xyz = "-0.275 ${-base_link_y/2-wheel_link_length/2} ${wheel_link_z}" rpy = "0 0 0" />
     <axis xyz ="1 0 0"/>
     <limit effort = "1000" velocity = "1000"/>
@@ -85,25 +101,21 @@
         <visual>
             <geometry>
-                <cylinder radius = "0.15" length = "0.05"/>
-            </geometry>
-            <origin xyz = " 0 0 0" rpy = "0 1.57 0"/>
+                <cylinder radius = "${wheel_link_radius}" length = "${wheel_link_length}"/>
+            </geometry>
+            <origin xyz = " 0 0 0" rpy = "0 1.570795 0"/>
             <material name = "white"/>
         </visual>
     <collision>
             <geometry>
-                <cylinder radius = "0.15" length = "0.05"/>
-            </geometry>
-            <origin xyz = " 0 0 0" rpy = "0 1.57 0"/>
-    </collision>
-    <inertial>
-         <origin xyz = " 0 0 0" rpy = "0 1.57 0"/>
-        <mass value= "0.25"/>
-        <inertia ixx = "100" ixy = "0" ixz = "0" iyy = "100" izz = "100" iyz = "0"/>
-    </inertial>
+                 <cylinder radius = "${wheel_link_radius}" length = "${wheel_link_length}"/>
+            </geometry>
+            <origin xyz = " 0 0 0" rpy = "0 1.570795 0"/>
+    </collision>
+  <xacro:inertial_wheel/>
     </link>
 <joint name = "left_back_wheel_joint" type = "continuous">
     <parent link = "base_link"/>
     <child link = "left_back_link"/>
-    <origin xyz = "0.275 -0.45 0" rpy = "0 0 0" />
+    <origin xyz = "0.275 ${base_link_y/2+wheel_link_length/2} ${wheel_link_z}" rpy = "0 0 0" />
     <axis xyz ="1 0 0"/>
     <limit effort = "1000" velocity = "1000"/>
@@ -113,25 +125,21 @@
         <visual>
             <geometry>
-                <cylinder radius = "0.15" length = "0.05"/>
-            </geometry>
-            <origin xyz = " 0 0 0" rpy = "0 1.57 0"/>
+               <cylinder radius = "${wheel_link_radius}" length = "${wheel_link_length}"/>
+            </geometry>
+            <origin xyz = " 0 0 0" rpy = "0 1.570795 0"/>
             <material name = "white"/>
         </visual>
      <collision>
             <geometry>
-                <cylinder radius = "0.15" length = "0.05"/>
-            </geometry>
-            <origin xyz = " 0 0 0" rpy = "0 1.57 0"/>
-    </collision>
-    <inertial>
-         <origin xyz = " 0 0 0" rpy = "0 1.57 0"/>
-        <mass value= "0.25"/>
-        <inertia ixx = "100" ixy = "0" ixz = "0" iyy = "100" izz = "100" iyz = "0"/>
-    </inertial>
+                <cylinder radius = "${wheel_link_radius}" length = "${wheel_link_length}"/>
+            </geometry>
+            <origin xyz = " 0 0 0" rpy = "0 1.570795 0"/>
+    </collision>
+    <xacro:inertial_wheel/>
     </link>
 <joint name = "right_back_wheel_joint" type = "continuous">
     <parent link = "base_link"/>
     <child link = "right_back_link"/>
-    <origin xyz = "-0.275 -0.45 0" rpy = "0 0 0" />
+    <origin xyz = "-0.275 ${base_link_y/2+wheel_link_length/2} ${wheel_link_z}" rpy = "0 0 0" />
     <axis xyz ="1 0 0"/>
     <limit effort = "1000" velocity = "1000"/>
@@ -141,20 +149,16 @@
         <visual>
             <geometry>
-                <cylinder radius = "0.15" length = "0.05"/>
-            </geometry>
-            <origin xyz = " 0 0 0" rpy = "0 1.57 0"/>
+                 <cylinder radius = "${wheel_link_radius}" length = "${wheel_link_length}"/>
+            </geometry>
+            <origin xyz = " 0 0 0" rpy = "0 1.570795 0"/>
             <material name = "white"/>
         </visual>
      <collision>
             <geometry>
-                <cylinder radius = "0.15" length = "0.05"/>
-            </geometry>
-            <origin xyz = " 0 0 0" rpy = "0 1.57 0"/>
-    </collision>
-    <inertial>
-         <origin xyz = " 0 0 0" rpy = "0 1.57 0"/>
-        <mass value= "0.25"/>
-        <inertia ixx = "100" ixy = "0" ixz = "0" iyy = "100" izz = "100" iyz = "0"/>
-    </inertial>
+                <cylinder radius = "${wheel_link_radius}" length = "${wheel_link_length}"/>
+            </geometry>
+            <origin xyz = " 0 0 0" rpy = "0 1.570795 0"/>
+    </collision>
+       <xacro:inertial_wheel/>
     </link>
 <joint name = "lidar_joint" type = "fixed">
@@ -163,45 +167,90 @@
     <origin xyz = "0 0.45 0.275" rpy = "0 0 0" />
 </joint>
-    <link name = "lidar_link">
-        <sensor type="lidar" name="lidar">
-            <laser>
-                <scan>
-                    <horizontal>
-                        <samples>1081</samples>
-                        <resolution>1.0</resolution>
-                    </horizontal>
-                </scan>
-                <range>
-                    <min>0.2</min>
-                    <max>30.0</max>
-                </range>
-            </laser>
-        </sensor>
-       <plugin name="lidar_plugin" filename="libgazebo_ros_laser.so">
-    <ros>
-        <namespace>lidar</namespace>
-        <remapping>scan:=/lidar/scan</remapping>
-        <param name="frame_id" value="lidar_link"/>
-    </ros>
+ <link name="lidar_link">
+    <visual>
+      <geometry>
+        <cylinder radius="0.05" length="0.1"/>
+      </geometry>
+      <material name="green"/>
+    </visual>
+    <collision>
+      <geometry>
+        <cylinder radius="0.05" length="0.1"/>
+      </geometry>
+    </collision>
+    <inertial>
+      <mass value="0.5"/>
+      <inertia ixx="0.01" ixy="0" ixz="0" iyy="0.01" iyz="0" izz="0.01"/>
+    </inertial>
+  </link>
+  <!-- Gazebo Plugin for Lidar -->
+  <gazebo reference="lidar_link">
+    <sensor name="lidar_sensor" type="ray">
+      <pose>0 0 0 0 0 0</pose>
+      <visualize>true</visualize>
+      <update_rate>10</update_rate>
+      <ray>
+        <scan>
+          <horizontal>
+            <samples>360</samples>
+            <resolution>1</resolution>
+            <min_angle>-3.14159</min_angle>
+            <max_angle>3.14159</max_angle>
+          </horizontal>
+        </scan>
+        <range>
+          <min>0.1</min>
+          <max>10.0</max>
+          <resolution>0.01</resolution>
+        </range>
+        <noise>
+          <type>gaussian</type>
+          <mean>0.0</mean>
+          <stddev>0.01</stddev>
+        </noise>
+      </ray>
+      <plugin name="lidar_plugin" filename="libgazebo_ros_ray_sensor.so">
+        <ros>
+          <namespace>lidar</namespace>
+          <remapping>~/out:=scan</remapping>
+        </ros>
+        <frame_name>lidar_link</frame_name>
+      </plugin>
+    </sensor>
+  </gazebo>
+<gazebo>
+<plugin name = 'skid_steer_drive' filename = 'libgazebo_ros_diff_drive.so'>
+<ros>
+<namespace></namespace>
+</ros>
+<num_wheel_pairs>2</num_wheel_pairs>
+<left_joint>left_front_wheel_joint</left_joint>
+<right_joint>right_back_wheel_joint</right_joint>
+<!--wheel_seperation value = "1.05"/!-->
+<wheel_seperation>1.05</wheel_seperation>
+<left_joint>left_back_wheel_joint</left_joint>
+<right_joint>right_front_wheel_joint</right_joint>
+<wheel_seperation>1.05</wheel_seperation>
+<!--wheel_seperation value = "1.05"/!-->
+<updateRate>$10</updateRate>
+<wheel_diameter>0.15</wheel_diameter>
+<wheel_diameter>0.15</wheel_diameter>
+<max_wheel_torque>1000</max_wheel_torque>
+<max_wheel_acceleration>5.0</max_wheel_acceleration>
+<commandTopic>cmd_vel</commandTopic>
+<odometryTopic>odom</odometryTopic>
+<odometryFrame>odom</odometryFrame>
+ <robotBaseFrame>base_link</robotBaseFrame>
+  <odometrySource>1</odometrySource>
+  <publishOdom>true</publishOdom>
+  <publishWheelJointState>true</publishWheelJointState>
+<publish_odom>true</publish_odom>
+<publish_odom_tf>true</publish_odom_tf>
+<publish_wheel_tf>true</publish_wheel_tf>
+<odom_publish_frequency>1</odom_publish_frequency>
+<odometry_frame>odom</odometry_frame>
+<robot_base_frame>left_front_link</robot_base_frame>
 </plugin>
-        <visual>
-            <geometry>
-                <box size = " 0.1 0.1 0.05 "/>
-            </geometry>
-            <origin xyz = " 0 0 0" rpy = "0 0 0"/>
-            <material name = "red"/>
-        </visual>
-     <collision>
-            <geometry>
-                <box size = " 0.1 0.1 0.05 "/>
-            </geometry>
-            <origin xyz = " 0 0 0" rpy = "0 0 0"/>
-    </collision>
-    <inertial>
-         <origin xyz = " 0 0 0" rpy = "0 0 0"/>
-        <mass value= "0.25"/>
-        <inertia ixx = "100" ixy = "0" ixz = "0" iyy = "100" izz = "100" iyz = "0"/>
-    </inertial>
-    </link>
+</gazebo>
 <joint name = "imu_joint" type = "fixed">
     <parent link = "base_link"/>
@@ -209,158 +258,157 @@
     <origin xyz = "0 -0.45 0.275" rpy = "0 0 0" />
 </joint>
-    <link name = "imu_link">
-         <sensor type="imu" name="imu">
-            <imu>
-                <update_rate>100.0</update_rate>
-                <raw>true</raw>
-                <frame_id>imu_link</frame_id>
-            </imu>
-        </sensor>
-        <plugin name="imu_plugin" filename="libgazebo_ros_imu.so">
-    <ros>
-        <namespace>imu</namespace>
-        <remapping>imu/data:=/imu/data</remapping>
-        <param name="frame_id" value="imu_link"/>
-    </ros>
-</plugin>
-        <visual>
-            <geometry>
-                <box size = " 0.1 0.1 0.05 "/>
-            </geometry>
-            <origin xyz = " 0 0 0" rpy = "0 0 0"/>
-            <material name = "blue"/>
-        </visual>
-    <collision>
-            <geometry>
-                <box size = " 0.1 0.1 0.05 "/>
-            </geometry>
-            <origin xyz = " 0 0 0" rpy = "0 0 0"/>
-    </collision>
-    <inertial>
-         <origin xyz = " 0 0 0" rpy = "0 0 0"/>
-        <mass value= "0.25"/>
-        <inertia ixx = "100" ixy = "0" ixz = "0" iyy = "100" izz = "100" iyz = "0"/>
-    </inertial>
-    </link>
+  <!-- IMU Link -->
+  <link name="imu_link">
+    <visual>
+      <geometry>
+        <cylinder radius="0.05" length="0.04"/>
+      </geometry>
+       <origin xyz="0 0 0" rpy="0 0 0"/>
+      <material name="black">
+        <color rgba="0 1 0 1"/>
+      </material>
+    </visual>
+    <collision>
+      <geometry>
+        <cylinder radius="0.05" length="0.04"/>
+      </geometry>
+    </collision>
+</link>
+  <gazebo reference="imu_link">
+    <sensor name="imu_sensor" type="imu">
+      <always_on>true</always_on>
+      <update_rate>10.0</update_rate>
+      <plugin name="imu_controller" filename="libgazebo_ros_imu_sensor.so">
+        <ros>
+          <remapping>imu_controller/out:=imu</remapping>
+        </ros>
+        <frame_name>imu_link</frame_name>
+      </plugin>
+    </sensor>
+    <material>Gazebo/Grey</material>
+  </gazebo>
     <!-- GPS Sensor -->
-    <link name="gps_link">
-        <plugin name="gps_plugin" filename="libgazebo_ros_gps.so">
-    <ros>
-        <namespace>gps</namespace>
-        <remapping>fix:=/gps/fix</remapping>
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