Commit message: Report added with OA partial done

File: ROS_Tasks/Obstacle_Avoidance/rover/model/rover.xacro (robot description, xacro)
@@ -2,7 +2,7 @@
 <robot xmlns:xacro="http://www.ros.org/wiki/xacro" name= "rover">
 <xacro:property name = "base_link_x" value = "0.5"/>
-<xacro:property name = "base_link_y" value = "1"/>
+<xacro:property name = "base_link_y" value = "0.5"/>
 <xacro:property name = "base_link_z" value = "0.25"/>
-<xacro:property name = "wheel_link_radius" value = "0.15"/>
+<xacro:property name = "wheel_link_radius" value = "0.05"/>
 <xacro:property name = "wheel_link_length" value = "0.05"/>
 <xacro:property name = "wheel_link_z" value = "0.075"/>
@@ -47,5 +47,5 @@
         <visual>
             <geometry>
-                <box size = "${base_link_x} ${base_link_y} ${base_link_z}"/>
+                <box size = "${base_link_x} ${base_link_x} ${base_link_z}"/>
             </geometry>
             <origin xyz = " 0 0 0.125" rpy = "0 0 0"/>
@@ -71,5 +71,5 @@
     <parent link = "base_link"/>
     <child link = "left_front_link"/>
-    <origin xyz = "0.275 ${-base_link_y/2-wheel_link_length/2} ${wheel_link_z}" rpy = "0 0 0" />
+    <origin xyz = "0.275 ${-base_link_x/2-wheel_link_length/2+0.1} ${wheel_link_z}" rpy = "0 0 0" />
     <axis xyz ="1 0 0"/>
     <limit effort = "1000" velocity = "1000"/>
@@ -95,5 +95,5 @@
     <parent link = "base_link"/>
     <child link = "right_front_link"/>
-    <origin xyz = "-0.275 ${-base_link_y/2-wheel_link_length/2} ${wheel_link_z}" rpy = "0 0 0" />
+    <origin xyz = "-0.275 ${-base_link_x/2-wheel_link_length/2+0.1} ${wheel_link_z}" rpy = "0 0 0" />
     <axis xyz ="1 0 0"/>
     <limit effort = "1000" velocity = "1000"/>
@@ -119,5 +119,5 @@
     <parent link = "base_link"/>
     <child link = "left_back_link"/>
-    <origin xyz = "0.275 ${base_link_y/2+wheel_link_length/2} ${wheel_link_z}" rpy = "0 0 0" />
+    <origin xyz = "0.275 ${base_link_x/2+wheel_link_length/2-0.1} ${wheel_link_z}" rpy = "0 0 0" />
     <axis xyz ="1 0 0"/>
     <limit effort = "1000" velocity = "1000"/>
@@ -143,5 +143,5 @@
     <parent link = "base_link"/>
     <child link = "right_back_link"/>
-    <origin xyz = "-0.275 ${base_link_y/2+wheel_link_length/2} ${wheel_link_z}" rpy = "0 0 0" />
+    <origin xyz = "-0.275 ${base_link_x/2+wheel_link_length/2-0.1} ${wheel_link_z}" rpy = "0 0 0" />
     <axis xyz ="1 0 0"/>
     <limit effort = "1000" velocity = "1000"/>
@@ -167,5 +167,5 @@
     <parent link = "base_link"/>
     <child link = "lidar_link"/>
-    <origin xyz = "0 0.45 0.275" rpy = "0 0 0" />
+    <origin xyz = "0 0.125 0.275" rpy = "0 0 0" />
 </joint>
  <link name="lidar_link">
@@ -186,40 +186,4 @@
     </inertial>
   </link>
-  <!-- Gazebo Plugin for Lidar -->
- <!-- <gazebo reference="lidar_link">
-    <sensor name="lidar" type="ray">
-      <pose>0 0 0 0 0 0 0</pose>
-      <always_on>true</always_on>
-      <visualize>true</visualize>
-      <update_rate>10</update_rate> -->
-      <!-- <ray>
-        <scan>
-          <horizontal>
-            <samples>360</samples>
-            <resolution>1.00000</resolution>
-            <min_angle>-1.57</min_angle>
-            <max_angle>1.57</max_angle>
-          </horizontal>
-        </scan>
-        <range>
-          <min>0.1</min>
-          <max>10</max>
-          <resolution>0.01</resolution>
-        </range>
-        <noise>
-          <type>gaussian</type>
-          <mean>0.0</mean>
-          <stddev>0.01</stddev>
-        </noise>
-      </ray> -->
-      <!-- <plugin name="scan" filename="libgazebo_ros_ray_sensor.so">
-        <ros>
-          <remapping>~/out:=scan</remapping>
-        </ros>
-        <output_type>sensor_msgs/LaserScan</output_type>
-        <frame_name>lidar_link</frame_name>
-      </plugin>
-    </sensor>
-  </gazebo> -->
  <gazebo reference="lidar_link">
     <sensor name="lidar" type="ray">
@@ -270,6 +234,6 @@
 <wheel_separation>1.05</wheel_separation>
 <updateRate>$10</updateRate>
-<wheel_diameter>0.15</wheel_diameter>
-<wheel_diameter>0.15</wheel_diameter>
+<wheel_diameter>0.1</wheel_diameter>
+<wheel_diameter>0.1</wheel_diameter>
 <max_wheel_torque>2000</max_wheel_torque>
 <max_wheel_acceleration>5.0</max_wheel_acceleration>
@@ -292,5 +256,5 @@
     <parent link = "base_link"/>
     <child link = "imu_link"/>
-    <origin xyz = "0 -0.45 0.275" rpy = "1.57 0 -3.14" />
+    <origin xyz = "0 -0.125 0.275" rpy = "1.57 0 -3.14" />
 </joint>
   <!-- IMU Link -->
